File: Hardware/arktika-fpga/arktika-fpga/Usb-and-prog.sch (KiCad schematic (older format))
At the start: 42 parts

Commit message: Updated eeprom info in component search, added missing bp cap to eeprom
Parts:
- removed UUP2: 93LCxxB, symbol Memory_EEPROM:93LCxxB
- added CUP9: 0.1u, symbol Device:C
- added UUP2: 93LC56B/OT, Package_TO_SOT_SMD:SOT-23-6, symbol Memory_EEPROM:93LCxxBxxOT
- renumbered CUP9 to CUP10
Connections:
- net EECLK: now also UUP2.4 (CLK)
- net EECS: now also UUP2.5 (CS)
- net EEDATA: now also UUP2.3 (DI)
- net GND: now also CUP9.2, UUP2.2 (GND)
- net VCC3V3_USB: now also CUP9.1, UUP2.6 (VCC)
- net at RUP7.2: now also UUP2.1 (DO)
Other:
- moved on the sheet: RUP7
Changed lines of the file:
@@
 $EndComp
 $Comp
-L Device:C CUP9
+L Device:C CUP10
 U 1 1 5F5400D2
 P 10700 4600
-F 0 "CUP9" H 10815 4646 50  0000 L CNN
+F 0 "CUP10" H 10815 4646 50  0000 L CNN
 F 1 "0.1u" H 10815 4555 50  0000 L CNN
 F 2 "Capacitors_SMD:C_0603" H 10738 4450 50  0001 C CNN
@@
 Wire Wire Line
 	1000 4200 1200 4200
-$Comp
-L Memory_EEPROM:93LCxxB UUP2
-U 1 1 5F64E466
-P 1800 6350
-F 0 "UUP2" H 1550 6600 50  0000 C CNN
-F 1 "93LCxxB" H 2000 6100 50  0000 C CNN
-F 2 "" H 1800 6350 50  0001 C CNN
-F 3 "http://ww1.microchip.com/downloads/en/DeviceDoc/20001749K.pdf" H 1800 6350 50  0001 C CNN
-	1    1800 6350
-	1    0    0    -1
-$EndComp
 Text Label 1800 5850 0    50   ~ 0
 VCC3V3_USB
@@
 	1    0    0    -1
 $EndComp
-$Comp
-L Device:R_US R?
-U 1 1 5F650447
-P 2400 6600
-AR Path="/5F650447" Ref="R?"  Part="1"
-AR Path="/5F3E98C5/5F650447" Ref="R?"  Part="1"
-AR Path="/5F415705/5F650447" Ref="RUP7"  Part="1"
-F 0 "RUP7" V 2300 6500 50  0000 C CNN
-F 1 "2.2k" V 2300 6700 50  0000 C CNN
-F 2 "Resistors_SMD:R_0603" V 2440 6590 50  0001 C CNN
-F 3 "~" H 2400 6600 50  0001 C CNN
-	1    2400 6600
-	0    1    -1   0
-$EndComp
-Wire Wire Line
-	2650 6350 2650 6600
-Wire Wire Line
-	2650 6600 2550 6600
-Wire Wire Line
-	2250 6600 2200 6600
-Wire Wire Line
-	2200 6600 2200 6450
 Text Label 2350 6350 0    50   ~ 0
 EEDATA
@@
 Wire Wire Line
 	2200 6250 2700 6250
-Wire Wire Line
-	2200 6350 2650 6350
-Connection ~ 2650 6350
 $Comp
 L Device:R_US R?
@@
 	-1   0    0    -1
 $EndComp
-Wire Wire Line
-	2650 6350 3000 6350
 Text Label 2850 5850 0    50   ~ 0
 VCC3V3_USB
@@
 VCC3V3_USB
 Wire Wire Line
-	950  5850 950  5950
+	950  5850 950  5900
 Wire Wire Line
 	950  6250 1400 6250
@@
 Connection ~ 5350 4400
 Wire Wire Line
-	1800 6650 1800 6750
+	1800 6650 1800 6700
 Wire Wire Line
 	1300 3400 1300 3450
@@
 Wire Wire Line
 	5350 4300 5800 4300
+$Comp
+L Memory_EEPROM:93LCxxBxxOT UUP2
+U 1 1 5F29EF92
+P 1800 6350
+F 0 "UUP2" H 1550 6600 50  0000 C CNN
+F 1 "93LC56B/OT" H 1450 6100 50  0000 C CNN
+F 2 "Package_TO_SOT_SMD:SOT-23-6" H 1800 6350 50  0001 C CNN
+F 3 "http://ww1.microchip.com/downloads/en/DeviceDoc/20001749K.pdf" H 1800 6350 50  0001 C CNN
+	1    1800 6350
+	1    0    0    -1
+$EndComp
+$Comp
+L Device:R_US R?
+U 1 1 5F650447
+P 2400 6450
+AR Path="/5F650447" Ref="R?"  Part="1"
+AR Path="/5F3E98C5/5F650447" Ref="R?"  Part="1"
+AR Path="/5F415705/5F650447" Ref="RUP7"  Part="1"
+F 0 "RUP7" V 2300 6350 50  0000 C CNN
+F 1 "2.2k" V 2300 6550 50  0000 C CNN
+F 2 "Resistors_SMD:R_0603" V 2440 6440 50  0001 C CNN
+F 3 "~" H 2400 6450 50  0001 C CNN
+	1    2400 6450
+	0    1    -1   0
+$EndComp
+Wire Wire Line
+	2200 6350 2700 6350
+Wire Wire Line
+	2200 6450 2250 6450
+Wire Wire Line
+	2550 6450 2700 6450
+Wire Wire Line
+	2700 6450 2700 6350
+Connection ~ 2700 6350
+Wire Wire Line
+	2700 6350 3000 6350
+$Comp
+L Device:C CUP9
+U 1 1 5F2BFCBB
+P 650 6450
+F 0 "CUP9" H 765 6496 50  0000 L CNN
+F 1 "0.1u" H 765 6405 50  0000 L CNN
+F 2 "" H 688 6300 50  0001 C CNN
+F 3 "~" H 650 6450 50  0001 C CNN
+	1    650  6450
+	1    0    0    -1
+$EndComp
+Wire Wire Line
+	950  5900 650  5900
+Wire Wire Line
+	650  5900 650  6300
+Connection ~ 950  5900
+Wire Wire Line
+	950  5900 950  5950
+Wire Wire Line
+	650  6600 650  6700
+Wire Wire Line
+	650  6700 1800 6700
+Connection ~ 1800 6700
+Wire Wire Line
+	1800 6700 1800 6750
 $EndSCHEMATC
