File: Hardware/arktika-fpga/arktika-fpga/FPGA_PERIPHS.sch (KiCad schematic (older format))
At the start: 28 parts

Commit message: Misc changes and fixes
Parts:
- added BPER1: Buzzer, symbol Device:Buzzer
- gave numbers to parts that had none: 1
Connections:
- net labels added: Buzzer
- wire segments 203 -> 206
Changed lines of the file:
@@
 $EndDescr
 $Comp
-L Analog_ADC:MCP3204 U?
+L Analog_ADC:MCP3204 UPER2
 U 1 1 5F72040D
 P 8950 5000
-F 0 "U?" H 9400 5450 50  0000 C CNN
+F 0 "UPER2" H 9400 5450 50  0000 C CNN
 F 1 "MCP3204" H 9250 5350 50  0000 C CNN
 F 2 "" H 9850 4700 50  0001 C CNN
@@
 Connection ~ 2750 950
 $Comp
-L power:GND #PWR?
+L power:GND #PWR0147
 U 1 1 5F729246
 P 2500 1250
-F 0 "#PWR?" H 2500 1000 50  0001 C CNN
+F 0 "#PWR0147" H 2500 1000 50  0001 C CNN
 F 1 "GND" H 2505 1077 50  0000 C CNN
 F 2 "" H 2500 1250 50  0001 C CNN
@@
 	1800 950  2250 950
 $Comp
-L power:GND #PWR?
+L power:GND #PWR0148
 U 1 1 5F72E759
 P 2500 1900
-F 0 "#PWR?" H 2500 1650 50  0001 C CNN
+F 0 "#PWR0148" H 2500 1650 50  0001 C CNN
 F 1 "GND" H 2505 1727 50  0000 C CNN
 F 2 "" H 2500 1900 50  0001 C CNN
@@
 	4350 1700 4650 1700
 $Comp
-L power:GND #PWR?
+L power:GND #PWR0149
 U 1 1 5F736641
 P 3850 3700
-F 0 "#PWR?" H 3850 3450 50  0001 C CNN
+F 0 "#PWR0149" H 3850 3450 50  0001 C CNN
 F 1 "GND" H 3855 3527 50  0000 C CNN
 F 2 "" H 3850 3700 50  0001 C CNN
@@
 AR Path="/5F751C99" Ref="#PWR?"  Part="1"
 AR Path="/5F3E98C5/5F751C99" Ref="#PWR?"  Part="1"
-AR Path="/5F72015E/5F751C99" Ref="#PWR?"  Part="1"
-F 0 "#PWR?" H 950 2050 50  0001 C CNN
+AR Path="/5F72015E/5F751C99" Ref="#PWR0150"  Part="1"
+F 0 "#PWR0150" H 950 2050 50  0001 C CNN
 F 1 "GND" H 950 2150 50  0000 C CNN
 F 2 "" H 950 2300 50  0001 C CNN
@@
 	3750 950  3850 950
 $Comp
-L power:GND #PWR?
+L power:GND #PWR0151
 U 1 1 5F27FA98
 P 3250 5950
-F 0 "#PWR?" H 3250 5700 50  0001 C CNN
+F 0 "#PWR0151" H 3250 5700 50  0001 C CNN
 F 1 "GND" H 3255 5777 50  0000 C CNN
 F 2 "" H 3250 5950 50  0001 C CNN
@@
 $EndComp
 $Comp
-L power:GND #PWR?
+L power:GND #PWR0152
 U 1 1 5F2089AF
 P 1650 5950
-F 0 "#PWR?" H 1650 5700 50  0001 C CNN
+F 0 "#PWR0152" H 1650 5700 50  0001 C CNN
 F 1 "GND" H 1655 5777 50  0000 C CNN
 F 2 "" H 1650 5950 50  0001 C CNN
@@
 AR Path="/5F21FDC0" Ref="#PWR?"  Part="1"
 AR Path="/5F3E98C5/5F21FDC0" Ref="#PWR?"  Part="1"
-AR Path="/5F72015E/5F21FDC0" Ref="#PWR?"  Part="1"
-F 0 "#PWR?" H 2100 2500 50  0001 C CNN
+AR Path="/5F72015E/5F21FDC0" Ref="#PWR0153"  Part="1"
+F 0 "#PWR0153" H 2100 2500 50  0001 C CNN
 F 1 "GND" H 2100 2600 50  0000 C CNN
 F 2 "" H 2100 2750 50  0001 C CNN
@@
 Text Label 10150 5500 1    50   ~ 0
 ADC
+Text HLabel 1250 7100 0    50   Input ~ 0
+PUSH_BTNS
 Text HLabel 1250 7200 0    50   Input ~ 0
+SWITCHES
+Text HLabel 1250 7300 0    50   Input ~ 0
+LEDS
+Text HLabel 1250 7400 0    50   Input ~ 0
+ADC
+Text Label 1350 7100 0    50   ~ 0
 PUSH_BTNS
-Text HLabel 1250 7300 0    50   Input ~ 0
+Text Label 1350 7200 0    50   ~ 0
 SWITCHES
-Text HLabel 1250 7400 0    50   Input ~ 0
+Text Label 1350 7300 0    50   ~ 0
 LEDS
-Text HLabel 1250 7500 0    50   Input ~ 0
+Text Label 1350 7400 0    50   ~ 0
 ADC
-Text Label 1350 7200 0    50   ~ 0
-PUSH_BTNS
-Text Label 1350 7300 0    50   ~ 0
-SWITCHES
-Text Label 1350 7400 0    50   ~ 0
-LEDS
-Text Label 1350 7500 0    50   ~ 0
-ADC
+Wire Bus Line
+	1250 7100 1800 7100
 Wire Bus Line
 	1250 7200 1800 7200
@@
 Wire Bus Line
 	1250 7400 1800 7400
-Wire Bus Line
-	1250 7500 1800 7500
 Entry Wire Line
 	4650 1200 4750 1300
@@
 Text Label 4750 2100 1    50   ~ 0
 UART
-Text HLabel 1250 7600 0    50   Input ~ 0
+Text HLabel 1250 7500 0    50   Input ~ 0
 UART
 Wire Bus Line
-	1250 7600 1800 7600
-Text Label 1350 7600 0    50   ~ 0
+	1250 7500 1800 7500
+Text Label 1350 7500 0    50   ~ 0
 UART
 Text Label 4550 4200 0    50   ~ 0
@@
 	4700 5700 5050 5700
 $Comp
-L power:GND #PWR?
+L power:GND #PWR0154
 U 1 1 5F226137
 P 5600 5750
-F 0 "#PWR?" H 5600 5500 50  0001 C CNN
+F 0 "#PWR0154" H 5600 5500 50  0001 C CNN
 F 1 "GND" H 5605 5577 50  0000 C CNN
 F 2 "" H 5600 5750 50  0001 C CNN
@@
 Wire Wire Line
 	3250 5850 3300 5850
-Text HLabel 1250 7100 0    50   Input ~ 0
+Text HLabel 1250 7000 0    50   Input ~ 0
 VCC3V3
-Text Label 1350 7100 0    50   ~ 0
+Text Label 1350 7000 0    50   ~ 0
 VCC3V3
 Wire Wire Line
-	1250 7100 1800 7100
+	1250 7000 1800 7000
 Text Label 1550 4350 1    50   ~ 0
 VCC3V3
@@
 Maybe find bridge with a easier package to solder. But also cheap\n
 $Comp
-L power:GND #PWR?
+L power:GND #PWR0155
 U 1 1 5F6F2DE0
 P 8900 5600
-F 0 "#PWR?" H 8900 5350 50  0001 C CNN
+F 0 "#PWR0155" H 8900 5350 50  0001 C CNN
 F 1 "GND" H 8905 5427 50  0000 C CNN
 F 2 "" H 8900 5600 50  0001 C CNN
@@
 Wire Wire Line
 	1650 1600 2250 1600
+$Comp
+L Device:Buzzer BPER1
+U 1 1 5F25EF58
+P 3400 7250
+F 0 "BPER1" H 3552 7279 50  0000 L CNN
+F 1 "Buzzer" H 3552 7188 50  0000 L CNN
+F 2 "" V 3375 7350 50  0001 C CNN
+F 3 "~" V 3375 7350 50  0001 C CNN
+	1    3400 7250
+	1    0    0    -1
+$EndComp
+$Comp
+L power:GND #PWR0156
+U 1 1 5F25F55A
+P 3300 7350
+F 0 "#PWR0156" H 3300 7100 50  0001 C CNN
+F 1 "GND" H 3305 7177 50  0000 C CNN
+F 2 "" H 3300 7350 50  0001 C CNN
+F 3 "" H 3300 7350 50  0001 C CNN
+	1    3300 7350
+	1    0    0    -1
+$EndComp
+Text HLabel 1250 7600 0    50   Input ~ 0
+Buzzer
+Wire Wire Line
+	1250 7600 1800 7600
+Text Label 1350 7600 0    50   ~ 0
+Buzzer
+Text Label 2900 7150 0    50   ~ 0
+Buzzer
+Wire Wire Line
+	2900 7150 3300 7150
+Text HLabel 1250 6600 0    50   Input ~ 0
+GND
+$Comp
+L power:GND #PWR?
+U 1 1 5F2D68F6
+P 1550 6600
+AR Path="/5F2D68F6" Ref="#PWR?"  Part="1"
+AR Path="/5F3E98C5/5F2D68F6" Ref="#PWR?"  Part="1"
+AR Path="/5F72015E/5F2D68F6" Ref="#PWR0157"  Part="1"
+F 0 "#PWR0157" H 1550 6350 50  0001 C CNN
+F 1 "GND" H 1550 6450 50  0000 C CNN
+F 2 "" H 1550 6600 50  0001 C CNN
+F 3 "" H 1550 6600 50  0001 C CNN
+	1    1550 6600
+	1    0    0    -1
+$EndComp
+Wire Wire Line
+	1550 6600 1250 6600
 Wire Bus Line
 	7850 5000 7850 5500

Commit message: Addded new hybrid crystal footprint, fixed missing footprints, created layout file for testing
Parts:
- BPER1: footprint (none) -> Buzzers_Beepers:Buzzer_12x9.5RM7.6
- CPER1, CPER2, CPER3, CPER4: footprint Capacitors_SMD:C_0603 -> Capacitors_SMD:C_0603_HandSoldering
- D0, D1, D2, D3, D4, D5, D6, D7: footprint (none) -> LEDs:LED_0603_HandSoldering
- DUSB2: footprint Package_TO_SOT_SMD:SOT-143 -> TO_SOT_Packages_SMD:SOT-143
- FUSB2: footprint (none) -> Fuses:Fuse_1812_4532Metric
- PSH0, PSH1, PSH2, PSH3: footprint (none) -> Buttons_Switches_SMD:SW_SPST_PTS645
- RPER1: footprint Resistors_SMD:R_0603 -> Resistors_SMD:R_0603_HandSoldering
- RPER2, RPER3, RPER4, RPER5, RPER6: footprint (none) -> Resistors_SMD:R_Array_Convex_4x0603
- SW[7..0]1: renamed from SW[7..0]; footprint (none) -> Buttons_Switches_SMD:SW_DIP_x8_W8.61mm_Slide_LowProfile
- UPER1: footprint Package_DFN_QFN:QFN-28-1EP_5x5mm_P0.5mm_EP3.35x3.35mm -> Housings_DFN_QFN:QFN-28-1EP_4x4mm_Pitch0.4mm
- UPER2: footprint (none) -> Housings_SOIC:SOIC-14_3.9x8.7mm_Pitch1.27mm
Changed lines of the file:
@@
 F 0 "UPER2" H 9400 5450 50  0000 C CNN
 F 1 "MCP3204" H 9250 5350 50  0000 C CNN
-F 2 "" H 9850 4700 50  0001 C CNN
+F 2 "Housings_SOIC:SOIC-14_3.9x8.7mm_Pitch1.27mm" H 9850 4700 50  0001 C CNN
 F 3 "http://ww1.microchip.com/downloads/en/DeviceDoc/21298c.pdf" H 9850 4700 50  0001 C CNN
 	1    8950 5000
@@
 F 0 "UPER1" H 4000 3700 50  0000 C CNN
 F 1 "CP2102N-A01-GQFN28" H 4400 3600 50  0000 C CNN
-F 2 "Package_DFN_QFN:QFN-28-1EP_5x5mm_P0.5mm_EP3.35x3.35mm" H 4300 1100 50  0001 L CNN
+F 2 "Housings_DFN_QFN:QFN-28-1EP_4x4mm_Pitch0.4mm" H 4300 1100 50  0001 L CNN
 F 3 "https://www.silabs.com/documents/public/data-sheets/cp2102n-datasheet.pdf" H 3900 1550 50  0001 C CNN
 	1    3850 2300
@@
 F 0 "CPER2" H 2865 1146 50  0000 L CNN
 F 1 "1u" H 2865 1055 50  0000 L CNN
-F 2 "Capacitors_SMD:C_0603" H 2788 950 50  0001 C CNN
+F 2 "Capacitors_SMD:C_0603_HandSoldering" H 2788 950 50  0001 C CNN
 F 3 "~" H 2750 1100 50  0001 C CNN
 	1    2750 1100
@@
 F 0 "CPER1" H 2365 1146 50  0000 L CNN
 F 1 "10u" H 2365 1055 50  0000 L CNN
-F 2 "Capacitors_SMD:C_0603" H 2288 950 50  0001 C CNN
+F 2 "Capacitors_SMD:C_0603_HandSoldering" H 2288 950 50  0001 C CNN
 F 3 "~" H 2250 1100 50  0001 C CNN
 	1    2250 1100
@@
 F 0 "CPER4" H 2865 1796 50  0000 L CNN
 F 1 "1u" H 2865 1705 50  0000 L CNN
-F 2 "Capacitors_SMD:C_0603" H 2788 1600 50  0001 C CNN
+F 2 "Capacitors_SMD:C_0603_HandSoldering" H 2788 1600 50  0001 C CNN
 F 3 "~" H 2750 1750 50  0001 C CNN
 	1    2750 1750
@@
 F 0 "CPER3" H 2365 1796 50  0000 L CNN
 F 1 "10u" H 2365 1705 50  0000 L CNN
-F 2 "Capacitors_SMD:C_0603" H 2288 1600 50  0001 C CNN
+F 2 "Capacitors_SMD:C_0603_HandSoldering" H 2288 1600 50  0001 C CNN
 F 3 "~" H 2250 1750 50  0001 C CNN
 	1    2250 1750
@@
 F 0 "RPER1" H 3218 1296 50  0000 L CNN
 F 1 "4.7k" H 3218 1205 50  0000 L CNN
-F 2 "Resistors_SMD:R_0603" V 3190 1240 50  0001 C CNN
+F 2 "Resistors_SMD:R_0603_HandSoldering" V 3190 1240 50  0001 C CNN
 F 3 "~" H 3150 1250 50  0001 C CNN
 	1    3150 1250
@@
 F 0 "DUSB2" H 2305 2546 50  0000 L CNN
 F 1 "SP0503BAHT" H 2305 2455 50  0000 L CNN
-F 2 "Package_TO_SOT_SMD:SOT-143" H 2325 2450 50  0001 L CNN
+F 2 "TO_SOT_Packages_SMD:SOT-143" H 2325 2450 50  0001 L CNN
 F 3 "http://www.littelfuse.com/~/media/files/littelfuse/technical%20resources/documents/data%20sheets/sp05xxba.pdf" H 2225 2625 50  0001 C CNN
 	1    2100 2500
@@
 F 0 "RPER4" H 3738 4496 50  0000 L CNN
 F 1 "1k" H 3738 4405 50  0000 L CNN
-F 2 "" V 3825 4450 50  0001 C CNN
+F 2 "Resistors_SMD:R_Array_Convex_4x0603" V 3825 4450 50  0001 C CNN
 F 3 "~" H 3550 4450 50  0001 C CNN
 	1    3550 4450
@@
 F 0 "RPER3" H 2550 4500 50  0000 L CNN
 F 1 "1k" H 2700 4400 50  0000 L CNN
-F 2 "" V 3325 4450 50  0001 C CNN
+F 2 "Resistors_SMD:R_Array_Convex_4x0603" V 3325 4450 50  0001 C CNN
 F 3 "~" H 3050 4450 50  0001 C CNN
 	1    3050 4450
@@
 F 0 "D7" V 4389 5282 50  0000 R CNN
 F 1 "LED" V 4298 5282 50  0000 R CNN
-F 2 "" H 4350 5400 50  0001 C CNN
+F 2 "LEDs:LED_0603_HandSoldering" H 4350 5400 50  0001 C CNN
 F 3 "~" H 4350 5400 50  0001 C CNN
 	1    4350 5400
@@
 F 0 "D5" V 5089 5282 50  0000 R CNN
 F 1 "LED" V 4998 5282 50  0000 R CNN
-F 2 "" H 5050 5400 50  0001 C CNN
+F 2 "LEDs:LED_0603_HandSoldering" H 5050 5400 50  0001 C CNN
 F 3 "~" H 5050 5400 50  0001 C CNN
 	1    5050 5400
@@
 F 0 "D4" V 5439 5282 50  0000 R CNN
 F 1 "LED" V 5348 5282 50  0000 R CNN
-F 2 "" H 5400 5400 50  0001 C CNN
+F 2 "LEDs:LED_0603_HandSoldering" H 5400 5400 50  0001 C CNN
 F 3 "~" H 5400 5400 50  0001 C CNN
 	1    5400 5400
@@
 F 0 "D3" V 5789 5282 50  0000 R CNN
 F 1 "LED" V 5698 5282 50  0000 R CNN
-F 2 "" H 5750 5400 50  0001 C CNN
+F 2 "LEDs:LED_0603_HandSoldering" H 5750 5400 50  0001 C CNN
 F 3 "~" H 5750 5400 50  0001 C CNN
 	1    5750 5400
@@
 F 0 "D2" V 6139 5282 50  0000 R CNN
 F 1 "LED" V 6048 5282 50  0000 R CNN
-F 2 "" H 6100 5400 50  0001 C CNN
+F 2 "LEDs:LED_0603_HandSoldering" H 6100 5400 50  0001 C CNN
 F 3 "~" H 6100 5400 50  0001 C CNN
 	1    6100 5400
@@
 F 0 "D1" V 6489 5282 50  0000 R CNN
 F 1 "LED" V 6398 5282 50  0000 R CNN
-F 2 "" H 6450 5400 50  0001 C CNN
+F 2 "LEDs:LED_0603_HandSoldering" H 6450 5400 50  0001 C CNN
 F 3 "~" H 6450 5400 50  0001 C CNN
 	1    6450 5400
@@
 F 0 "D0" V 6839 5282 50  0000 R CNN
 F 1 "LED" V 6748 5282 50  0000 R CNN
-F 2 "" H 6800 5400 50  0001 C CNN
+F 2 "LEDs:LED_0603_HandSoldering" H 6800 5400 50  0001 C CNN
 F 3 "~" H 6800 5400 50  0001 C CNN
 	1    6800 5400
@@
 F 0 "RPER5" H 5138 4796 50  0000 L CNN
 F 1 "660?" H 5138 4705 50  0000 L CNN
-F 2 "" V 5225 4750 50  0001 C CNN
+F 2 "Resistors_SMD:R_Array_Convex_4x0603" V 5225 4750 50  0001 C CNN
 F 3 "~" H 4950 4750 50  0001 C CNN
 	1    4950 4750
@@
 F 0 "RPER6" H 6538 4796 50  0000 L CNN
 F 1 "660?" H 6538 4705 50  0000 L CNN
-F 2 "" V 6625 4750 50  0001 C CNN
+F 2 "Resistors_SMD:R_Array_Convex_4x0603" V 6625 4750 50  0001 C CNN
 F 3 "~" H 6350 4750 50  0001 C CNN
 	1    6350 4750
@@
 L Device:R_Pack04 RPER2
 U 1 1 5F234827
-P 1600 4700
-F 0 "RPER2" H 1788 4746 50  0000 L CNN
-F 1 "1k" H 1788 4655 50  0000 L CNN
-F 2 "" V 1875 4700 50  0001 C CNN
-F 3 "~" H 1600 4700 50  0001 C CNN
-	1    1600 4700
-	1    0    0    -1
+P 1500 4700
+F 0 "RPER2" H 1688 4746 50  0000 L CNN
+F 1 "1k" H 1688 4655 50  0000 L CNN
+F 2 "Resistors_SMD:R_Array_Convex_4x0603" V 1775 4700 50  0001 C CNN
+F 3 "~" H 1500 4700 50  0001 C CNN
+	1    1500 4700
+	-1   0    0    -1
 $EndComp
 Wire Wire Line
@@
 	2500 1900 2750 1900
 $Comp
-L Switch:SW_DIP_x08 SW[7..0]
+L Switch:SW_DIP_x08 SW[7..0]1
 U 1 1 5F27896E
 P 3200 5550
-F 0 "SW[7..0]" V 3154 6080 50  0000 L CNN
+F 0 "SW[7..0]1" V 3154 6080 50  0000 L CNN
 F 1 "SW_DIP_x08" V 3245 6080 50  0000 L CNN
-F 2 "" H 3200 5550 50  0001 C CNN
+F 2 "Buttons_Switches_SMD:SW_DIP_x8_W8.61mm_Slide_LowProfile" H 3200 5550 50  0001 C CNN
 F 3 "~" H 3200 5550 50  0001 C CNN
 	1    3200 5550
@@
 F 0 "PSH0" V 2200 5552 50  0000 R CNN
 F 1 "SW_Push" V 2155 5552 50  0001 R CNN
-F 2 "" H 2200 5800 50  0001 C CNN
+F 2 "Buttons_Switches_SMD:SW_SPST_PTS645" H 2200 5800 50  0001 C CNN
 F 3 "~" H 2200 5800 50  0001 C CNN
 	1    2200 5600
@@
 F 0 "PSH1" V 1850 5552 50  0000 R CNN
 F 1 "SW_Push" V 1805 5552 50  0001 R CNN
-F 2 "" H 1850 5800 50  0001 C CNN
+F 2 "Buttons_Switches_SMD:SW_SPST_PTS645" H 1850 5800 50  0001 C CNN
 F 3 "~" H 1850 5800 50  0001 C CNN
 	1    1850 5600
@@
 F 0 "PSH2" V 1500 5552 50  0000 R CNN
 F 1 "SW_Push" V 1455 5552 50  0001 R CNN
-F 2 "" H 1500 5800 50  0001 C CNN
+F 2 "Buttons_Switches_SMD:SW_SPST_PTS645" H 1500 5800 50  0001 C CNN
 F 3 "~" H 1500 5800 50  0001 C CNN
 	1    1500 5600
@@
 F 0 "PSH3" V 1150 5552 50  0000 R CNN
 F 1 "SW_Push" V 1105 5552 50  0001 R CNN
-F 2 "" H 1150 5800 50  0001 C CNN
+F 2 "Buttons_Switches_SMD:SW_SPST_PTS645" H 1150 5800 50  0001 C CNN
 F 3 "~" H 1150 5800 50  0001 C CNN
 	1    1150 5600
@@
 F 0 "D6" V 4739 5282 50  0000 R CNN
 F 1 "LED" V 4648 5282 50  0000 R CNN
-F 2 "" H 4700 5400 50  0001 C CNN
+F 2 "LEDs:LED_0603_HandSoldering" H 4700 5400 50  0001 C CNN
 F 3 "~" H 4700 5400 50  0001 C CNN
 	1    4700 5400
@@
 F 0 "FUSB2" V 1303 1600 50  0000 C CNN
 F 1 "500mA?" V 1394 1600 50  0000 C CNN
-F 2 "" V 1430 1600 50  0001 C CNN
+F 2 "Fuses:Fuse_1812_4532Metric" V 1430 1600 50  0001 C CNN
 F 3 "~" H 1500 1600 50  0001 C CNN
 	1    1500 1600
@@
 F 0 "BPER1" H 3552 7279 50  0000 L CNN
 F 1 "Buzzer" H 3552 7188 50  0000 L CNN
-F 2 "" V 3375 7350 50  0001 C CNN
+F 2 "Buzzers_Beepers:Buzzer_12x9.5RM7.6" V 3375 7350 50  0001 C CNN
 F 3 "~" V 3375 7350 50  0001 C CNN
 	1    3400 7250

Commit message: Misc schematic changes. Preliminary layout almost complete
Parts:
- BPER1: symbol Device:Buzzer -> arktika-fpga-rescue:Buzzer-Device
- CPER1, CPER2, CPER3, CPER4: footprint Capacitors_SMD:C_0603_HandSoldering -> Capacitor_SMD:C_0603_1608Metric_Pad1.05x0.95mm_HandSolder; symbol Device:C -> arktika-fpga-rescue:C-Device
- D0, D1, D2, D3, D4, D5, D6, D7: footprint LEDs:LED_0603_HandSoldering -> LED_SMD:LED_0603_1608Metric_Pad1.05x0.95mm_HandSolder; symbol Device:LED -> arktika-fpga-rescue:LED-Device
- DUSB2: footprint TO_SOT_Packages_SMD:SOT-143 -> Package_TO_SOT_SMD:SOT-143; symbol Power_Protection:SP0503BAHT -> arktika-fpga-rescue:SP0503BAHT-Power_Protection
- FUSB2: footprint Fuses:Fuse_1812_4532Metric -> Fuse:Fuse_1812_4532Metric_Pad1.30x3.40mm_HandSolder; symbol Device:Fuse -> arktika-fpga-rescue:Fuse-Device
- JUSB2: symbol Connector:USB_B_Micro -> arktika-fpga-rescue:USB_B_Micro-Connector
- PSH0, PSH1, PSH2, PSH3: footprint Buttons_Switches_SMD:SW_SPST_PTS645 -> Button_Switch_SMD:SW_SPST_PTS645; symbol Switch:SW_Push -> arktika-fpga-rescue:SW_Push-Switch
- RPER1: footprint Resistors_SMD:R_0603_HandSoldering -> Resistor_SMD:R_0603_1608Metric_Pad1.05x0.95mm_HandSolder; symbol Device:R_US -> arktika-fpga-rescue:R_US-Device
- RPER2, RPER3, RPER4, RPER5, RPER6: footprint Resistors_SMD:R_Array_Convex_4x0603 -> Resistor_SMD:R_Array_Convex_4x0603; symbol Device:R_Pack04 -> arktika-fpga-rescue:R_Pack04-Device
- SW[7..0]1: footprint Buttons_Switches_SMD:SW_DIP_x8_W8.61mm_Slide_LowProfile -> Button_Switch_SMD:SW_DIP_SPSTx08_Slide_6.7x21.88mm_W8.61mm_P2.54mm_LowProfile; symbol Switch:SW_DIP_x08 -> arktika-fpga-rescue:SW_DIP_x08-Switch
- UPER1: footprint Housings_DFN_QFN:QFN-28-1EP_4x4mm_Pitch0.4mm -> Package_DFN_QFN:QFN-28-1EP_4x4mm_P0.4mm_EP2.6x2.6mm; symbol Interface_USB:CP2102N-A01-GQFN28 -> arktika-fpga-rescue:CP2102N-A01-GQFN28-Interface_USB
- UPER2: footprint Housings_SOIC:SOIC-14_3.9x8.7mm_Pitch1.27mm -> Package_SO:SOIC-14_3.9x8.7mm_P1.27mm; symbol Analog_ADC:MCP3204 -> arktika-fpga-rescue:MCP3204-Analog_ADC
Connections:
- net labels added: LED[0..7], PSH[0..3], SW[0..7], UART_RX, UART_TX
- net labels removed: ADC, LEDS, PUSH_BTNS, SWITCHES, UART
- wire segments 206 -> 202

Commit message: Added more IO
Parts:
- BPER1: footprint Buzzers_Beepers:Buzzer_12x9.5RM7.6 -> Connector_PinHeader_2.54mm:PinHeader_1x02_P2.54mm_Vertical
Changed lines of the file:
@@
 Wire Wire Line
 	1650 1600 2250 1600
-$Comp
-L arktika-fpga-rescue:Buzzer-Device BPER1
-U 1 1 5F25EF58
-P 3400 7250
-F 0 "BPER1" H 3552 7279 50  0000 L CNN
-F 1 "Buzzer" H 3552 7188 50  0000 L CNN
-F 2 "Buzzers_Beepers:Buzzer_12x9.5RM7.6" V 3375 7350 50  0001 C CNN
-F 3 "~" V 3375 7350 50  0001 C CNN
-	1    3400 7250
-	1    0    0    -1
-$EndComp
-$Comp
-L arktika-fpga-rescue:GND-power #PWR0156
-U 1 1 5F25F55A
-P 3300 7350
-F 0 "#PWR0156" H 3300 7100 50  0001 C CNN
-F 1 "GND" H 3305 7177 50  0000 C CNN
-F 2 "" H 3300 7350 50  0001 C CNN
-F 3 "" H 3300 7350 50  0001 C CNN
-	1    3300 7350
-	1    0    0    -1
-$EndComp
 Text HLabel 1250 7400 0    50   Input ~ 0
 Buzzer
@@
 Text Label 1350 7400 0    50   ~ 0
 Buzzer
-Text Label 2900 7150 0    50   ~ 0
-Buzzer
-Wire Wire Line
-	2900 7150 3300 7150
 Text HLabel 1250 6600 0    50   Input ~ 0
 GND
@@
 UART_TX
 Wire Bus Line
+	2450 4800 3450 4800
+Wire Bus Line
 	650  5150 2000 5150
 Wire Bus Line
-	2450 4800 3450 4800
-Wire Bus Line
 	4550 4200 6350 4200
+Wire Wire Line
+	2900 7150 3300 7150
+Text Label 2900 7150 0    50   ~ 0
+Buzzer
+$Comp
+L arktika-fpga-rescue:GND-power #PWR0156
+U 1 1 5F25F55A
+P 3300 7350
+F 0 "#PWR0156" H 3300 7100 50  0001 C CNN
+F 1 "GND" H 3305 7177 50  0000 C CNN
+F 2 "" H 3300 7350 50  0001 C CNN
+F 3 "" H 3300 7350 50  0001 C CNN
+	1    3300 7350
+	1    0    0    -1
+$EndComp
+$Comp
+L arktika-fpga-rescue:Buzzer-Device BPER1
+U 1 1 5F25EF58
+P 3400 7250
+F 0 "BPER1" H 3552 7279 50  0000 L CNN
+F 1 "Buzzer" H 3552 7188 50  0000 L CNN
+F 2 "Connector_PinHeader_2.54mm:PinHeader_1x02_P2.54mm_Vertical" V 3375 7350 50  0001 C CNN
+F 3 "~" V 3375 7350 50  0001 C CNN
+	1    3400 7250
+	1    0    0    -1
+$EndComp
 $EndSCHEMATC
